File: V9203.sch (KiCad schematic (older format))
At the start: 79 parts, among them J1 RJ45, J10 GS3, J4 Screw_Terminal_1x04, J6 CONN_01X09, J7 GS3, J8 GS3, U1 V9203, Y1 Crystal_GND24

Commit message: Laid out components so far pending ERC,routing and review
Parts:
- added LOGO2: LOGO, symbol LOGO
Connections:
- net +3V3: now also J10.1 (G1), R43.1; no longer C30.2, J10.3 (G3)
- net GND: now also C30.2, J10.3 (G3); no longer J10.1 (G1), R43.1
Changed lines of the file:
@@
 $EndComp
 $Comp
-L GND #PWR01
+L GND #PWR10
 U 1 1 58D7BD25
 P 4700 1350
-F 0 "#PWR01" H -100 -900 50  0001 C CNN
+F 0 "#PWR10" H -100 -900 50  0001 C CNN
 F 1 "GND" H 4705 1177 50  0000 C CNN
 F 2 "" H -100 -650 50  0001 C CNN
@@
 $EndComp
 $Comp
-L PWR_FLAG #FLG02
+L PWR_FLAG #FLG2
 U 1 1 58D7C0C0
 P 4700 1900
-F 0 "#FLG02" H -150 75  50  0001 C CNN
+F 0 "#FLG2" H -150 75  50  0001 C CNN
 F 1 "PWR_FLAG" V 4700 2028 50  0000 L CNN
 F 2 "" H -150 0   50  0001 C CNN
@@
 $EndComp
 $Comp
-L GND #PWR03
+L GND #PWR9
 U 1 1 58D7CCEA
 P 4050 2900
-F 0 "#PWR03" H -750 650 50  0001 C CNN
+F 0 "#PWR9" H -750 650 50  0001 C CNN
 F 1 "GND" V 4055 2772 50  0000 R CNN
 F 2 "" H -750 900 50  0001 C CNN
@@
 $EndComp
 $Comp
-L GND #PWR04
+L GND #PWR8
 U 1 1 58D7CDA6
 P 3900 2200
-F 0 "#PWR04" H -900 -50 50  0001 C CNN
+F 0 "#PWR8" H -900 -50 50  0001 C CNN
 F 1 "GND" H 3905 2027 50  0000 C CNN
 F 2 "" H -900 200 50  0001 C CNN
@@
 $EndComp
 $Comp
-L PWR_FLAG #FLG05
+L PWR_FLAG #FLG1
 U 1 1 58D7CE59
 P 3350 2700
-F 0 "#FLG05" H -1500 875 50  0001 C CNN
+F 0 "#FLG1" H -1500 875 50  0001 C CNN
 F 1 "PWR_FLAG" V 3350 2828 50  0000 L CNN
 F 2 "" H -1500 800 50  0001 C CNN
@@
 $EndComp
 $Comp
-L GND #PWR06
+L GND #PWR1
 U 1 1 58D7E932
 P 1550 2950
-F 0 "#PWR06" H -3250 700 50  0001 C CNN
+F 0 "#PWR1" H -3250 700 50  0001 C CNN
 F 1 "GND" V 1555 2822 50  0000 R CNN
 F 2 "" H -3250 950 50  0001 C CNN
@@
 $EndComp
 $Comp
-L GND #PWR07
+L GND #PWR2
 U 1 1 58D7EE20
 P 1550 3900
-F 0 "#PWR07" H -3250 1650 50  0001 C CNN
+F 0 "#PWR2" H -3250 1650 50  0001 C CNN
 F 1 "GND" V 1555 3772 50  0000 R CNN
 F 2 "" H -3250 1900 50  0001 C CNN
@@
 $EndComp
 $Comp
-L GND #PWR08
+L GND #PWR7
 U 1 1 58D7EE5B
 P 2550 3900
-F 0 "#PWR08" H -2250 1650 50  0001 C CNN
+F 0 "#PWR7" H -2250 1650 50  0001 C CNN
 F 1 "GND" V 2555 3772 50  0000 R CNN
 F 2 "" H -2250 1900 50  0001 C CNN
@@
 $EndComp
 $Comp
-L GND #PWR09
+L GND #PWR6
 U 1 1 58D7EE96
 P 2550 2950
-F 0 "#PWR09" H -2250 700 50  0001 C CNN
+F 0 "#PWR6" H -2250 700 50  0001 C CNN
 F 1 "GND" V 2555 2822 50  0000 R CNN
 F 2 "" H -2250 950 50  0001 C CNN
@@
 $EndComp
 $Comp
-L GND #PWR010
+L GND #PWR3
 U 1 1 58D8C933
 P 2000 5600
-F 0 "#PWR010" H -2800 3350 50  0001 C CNN
+F 0 "#PWR3" H -2800 3350 50  0001 C CNN
 F 1 "GND" H 2005 5427 50  0000 C CNN
 F 2 "" H -2800 3600 50  0001 C CNN
@@
 $EndComp
 $Comp
-L GND #PWR011
+L GND #PWR4
 U 1 1 58D8CC7A
 P 2000 6250
-F 0 "#PWR011" H -2800 4000 50  0001 C CNN
+F 0 "#PWR4" H -2800 4000 50  0001 C CNN
 F 1 "GND" H 2005 6077 50  0000 C CNN
 F 2 "" H -2800 4250 50  0001 C CNN
@@
 $EndComp
 $Comp
-L GND #PWR012
+L GND #PWR5
 U 1 1 58D8CE39
 P 2000 6900
-F 0 "#PWR012" H -2800 4650 50  0001 C CNN
+F 0 "#PWR5" H -2800 4650 50  0001 C CNN
 F 1 "GND" H 2005 6727 50  0000 C CNN
 F 2 "" H -2800 4900 50  0001 C CNN
@@
 $EndComp
 $Comp
-L GND #PWR013
+L GND #PWR11
 U 1 1 58D8D54A
 P 4700 5400
-F 0 "#PWR013" H -100 3150 50  0001 C CNN
+F 0 "#PWR11" H -100 3150 50  0001 C CNN
 F 1 "GND" H 4705 5227 50  0000 C CNN
 F 2 "" H -100 3400 50  0001 C CNN
@@
 $EndComp
 $Comp
-L GND #PWR014
+L GND #PWR14
 U 1 1 58EFA437
 P 8150 3900
-F 0 "#PWR014" H 3350 1650 50  0001 C CNN
+F 0 "#PWR14" H 3350 1650 50  0001 C CNN
 F 1 "GND" H 8155 3727 50  0000 C CNN
 F 2 "" H 3350 1900 50  0001 C CNN
@@
 $EndComp
 $Comp
-L GND #PWR015
+L GND #PWR12
 U 1 1 58EFBDC4
 P 5900 5400
-F 0 "#PWR015" H 1100 3150 50  0001 C CNN
+F 0 "#PWR12" H 1100 3150 50  0001 C CNN
 F 1 "GND" H 5905 5227 50  0000 C CNN
 F 2 "" H 1100 3400 50  0001 C CNN
@@
 $EndComp
 $Comp
-L PWR_FLAG #FLG016
+L PWR_FLAG #FLG3
 U 1 1 58EFD209
 P 5100 5700
-F 0 "#FLG016" H 250 3875 50  0001 C CNN
+F 0 "#FLG3" H 250 3875 50  0001 C CNN
 F 1 "PWR_FLAG" V 5100 5828 50  0000 L CNN
 F 2 "" H 250 3800 50  0001 C CNN
@@
 $EndComp
 $Comp
-L PWR_FLAG #FLG017
+L PWR_FLAG #FLG5
 U 1 1 58F50052
 P 9200 4550
-F 0 "#FLG017" H 4350 2725 50  0001 C CNN
+F 0 "#FLG5" H 4350 2725 50  0001 C CNN
 F 1 "PWR_FLAG" V 9200 4678 50  0000 L CNN
 F 2 "" H 4350 2650 50  0001 C CNN
@@
 V_CS
 $Comp
-L GND #PWR018
+L GND #PWR16
 U 1 1 58FE85DB
 P 10600 4500
-F 0 "#PWR018" H 5800 2250 50  0001 C CNN
+F 0 "#PWR16" H 5800 2250 50  0001 C CNN
 F 1 "GND" H 10605 4327 50  0000 C CNN
 F 2 "" H 5800 2500 50  0001 C CNN
@@
 	7600 4750 7600 4700
 $Comp
-L GND #PWR019
+L GND #PWR13
 U 1 1 5905C1C0
 P 7600 4750
-F 0 "#PWR019" H 2800 2500 50  0001 C CNN
+F 0 "#PWR13" H 2800 2500 50  0001 C CNN
 F 1 "GND" H 7605 4577 50  0000 C CNN
 F 2 "" H 2800 2750 50  0001 C CNN
@@
 Text Label 7500 5400 0    60   ~ 0
 DS
-Text GLabel 8850 5900 2    60   Input ~ 0
+Text GLabel 8700 5100 1    60   Input ~ 0
 +3V3
 $Comp
-L PWR_FLAG #FLG020
+L PWR_FLAG #FLG4
 U 1 1 5905FDEF
 P 8850 5700
-F 0 "#FLG020" H 4000 3875 50  0001 C CNN
+F 0 "#FLG4" H 4000 3875 50  0001 C CNN
 F 1 "PWR_FLAG" V 8850 5828 50  0000 L CNN
 F 2 "" H 4000 3800 50  0001 C CNN
@@
 $EndComp
 $Comp
-L GND #PWR021
+L GND #PWR15
 U 1 1 59060110
-P 8850 5100
-F 0 "#PWR021" H 4050 2850 50  0001 C CNN
-F 1 "GND" H 8855 4927 50  0000 C CNN
-F 2 "" H 4050 3100 50  0001 C CNN
-F 3 "" H 4050 3100 50  0001 C CNN
-	1    8850 5100
+P 8850 5900
+F 0 "#PWR15" H 4050 3650 50  0001 C CNN
+F 1 "GND" H 8855 5727 50  0000 C CNN
+F 2 "" H 4050 3900 50  0001 C CNN
+F 3 "" H 4050 3900 50  0001 C CNN
+	1    8850 5900
 	0    -1   -1   0
 $EndComp
+$Comp
+L LOGO LOGO2
+U 1 1 590551CB
+P 9950 5500
+F 0 "LOGO2" H 10000 5550 60  0001 C CNN
+F 1 "LOGO" H -150 252 60  0001 C CNN
+F 2 "" H -150 150 60  0001 C CNN
+F 3 "" H -150 150 60  0001 C CNN
+F 4 "Value" H 9950 5500 60  0001 C CNN "manf#"
+	1    9950 5500
+	1    0    0    -1
+$EndComp
 $EndSCHEMATC
